Commit message: feat: Added d435 to scout_mini
The scout_empty_world.launch file was modified to include intel d435

File: src/scout_mini_ros/scout_description/urdf/custom_description.urdf (robot description, URDF)
Before this commit: robot accessories, 4 links, 4 joints
Links:
- removed link t265_pose_frame
Joints:
- removed joint cam_link_t265
