Commit message: Feature Addition
Modify the scout model and spawn it in the chironix lab world with sensors and move base configured.

File: src/scout_mini_ros/scout/scout_description/urdf/custom_description.urdf (robot description, URDF)
Before this commit: robot accessories, 4 links, 4 joints
Links:
- removed link t265_pose_frame
Joints:
- removed joint cam_link_t265

File: src/scout_mini_ros/scout/scout_description/urdf/mini.urdf (robot description, URDF)
Before this commit: robot scout_mini, 14 links, 13 joints
Links:
- link t265_pose_frame: geometry visual mesh filename=package://realsense2_description/meshes/d415.stl
