Commit message: Feature Addition - Husky sim
Modify the husky model and spawn it in the chironix lab world with sensors and move base configured.

File: src/scout_mini_ros/husky/husky_description/urdf/husky.urdf.xacro (robot description, xacro)
@@ -39,4 +39,5 @@
   <xacro:include filename="$(find husky_description)/urdf/accessories/sick_lms1xx_mount.urdf.xacro"/>
   <xacro:include filename="$(find husky_description)/urdf/accessories/sensor_arch.urdf.xacro"/>
+  <xacro:include filename="$(find velodyne_description)/urdf/VLP-16.urdf.xacro"/>
   <xacro:property name="M_PI" value="3.14159"/>
   <!-- Base Size -->
@@ -117,6 +118,6 @@
   <xacro:husky_decorate />
   <xacro:if value="$(arg laser_enabled)">
-    <sick_lms1xx_mount prefix="base"/>
-    <sick_lms1xx frame="base_laser" topic="scan" robot_namespace="$(arg robot_namespace)"/>
+    <xacro:sick_lms1xx_mount prefix="base"/>
+    <xacro:sick_lms1xx frame="base_laser" topic="scan" robot_namespace="$(arg robot_namespace)"/>
     <joint name="laser_mount_joint" type="fixed">
       <origin xyz="$(arg laser_xyz)" rpy="$(arg laser_rpy)" />
@@ -183,3 +184,45 @@
   <!-- Optional custom includes. -->
   <xacro:include filename="$(arg urdf_extras)" />
+  <!-- Velodyne -->
+  <!-- <xacro:include filename="$(find velodyne_description)/urdf/VLP-16.urdf.xacro" />
+  <xacro:VLP-16 name="laser_scan" parent="base" ros_topic="base_scan/scan"
+      update_rate="20" min_angle="-1.57" max_angle="1.57" >
+        <origin xyz="${0.4 - 0.01 - 0.04} 0 0.3" rpy="0 0 0" />
+    </xacro:VLP-16>
+<joint name="laser_joint" type="fixed">
+        <origin xyz="${0.4 - 0.01 - 0.04} 0 0.3" rpy="0 0 0" />
+        <parent link="base_link" />
+        <child link="laser_link"/>
+    </joint>
+    <link name="laser_link">
+      <inertial>
+            <mass value="0.01" />
+            <origin xyz="0 0 0" />
+            <inertia ixx="0.001"  ixy="0.0"  ixz="0.0"
+            iyy="0.001"  iyz="0.0"
+                izz="0.001" />
+            </inertial>
+            <visual>
+                <origin xyz="0 0 0" rpy="0 0 0"/>
+                <geometry>
+                    <box size="0.05 0.05 0.1" />
+                </geometry>
+            </visual>
+            <collision>
+                <origin xyz="0 0 0" rpy="0 0 0"/>
+                <geometry>
+                    <box size="0.05 0.05 0.1" />
+                </geometry>
+            </collision>
+        </link> -->
+  <!--Velodyne and Velodyne Interface -->
+  <link name="velodyne_mount"/>
+  <joint name="velodyne_mount_joint" type="fixed">
+    <parent link="base_link"/>
+    <child link="velodyne_mount"/>
+    <origin xyz="0.1 0 0.17" rpy="0 0 0"/>
+  </joint>
+  <xacro:VLP-16 parent="velodyne_mount" name="velodyne" topic="/velodyne_points" hz="10" organize_cloud="true" samples="200" gpu="false">
+    <origin xyz="0 0 0" rpy="0 0 0" />
+  </xacro:VLP-16>
 </robot>

Commit message: Code clean up
Clean up the husky urdf file and disable the deafault 2D laser scan.

File: src/scout_mini_ros/husky/husky_description/urdf/husky.urdf.xacro (robot description, xacro)
@@ -185,37 +185,4 @@
   <xacro:include filename="$(arg urdf_extras)" />
   <!-- Velodyne -->
-  <!-- <xacro:include filename="$(find velodyne_description)/urdf/VLP-16.urdf.xacro" />
-  <xacro:VLP-16 name="laser_scan" parent="base" ros_topic="base_scan/scan"
-      update_rate="20" min_angle="-1.57" max_angle="1.57" >
-        <origin xyz="${0.4 - 0.01 - 0.04} 0 0.3" rpy="0 0 0" />
-    </xacro:VLP-16>
-<joint name="laser_joint" type="fixed">
-        <origin xyz="${0.4 - 0.01 - 0.04} 0 0.3" rpy="0 0 0" />
-        <parent link="base_link" />
-        <child link="laser_link"/>
-    </joint>
-    <link name="laser_link">
-      <inertial>
-            <mass value="0.01" />
-            <origin xyz="0 0 0" />
-            <inertia ixx="0.001"  ixy="0.0"  ixz="0.0"
-            iyy="0.001"  iyz="0.0"
-                izz="0.001" />
-            </inertial>
-            <visual>
-                <origin xyz="0 0 0" rpy="0 0 0"/>
-                <geometry>
-                    <box size="0.05 0.05 0.1" />
-                </geometry>
-            </visual>
-            <collision>
-                <origin xyz="0 0 0" rpy="0 0 0"/>
-                <geometry>
-                    <box size="0.05 0.05 0.1" />
-                </geometry>
-            </collision>
-        </link> -->
-  <!--Velodyne and Velodyne Interface -->
-  <link name="velodyne_mount"/>
   <joint name="velodyne_mount_joint" type="fixed">
     <parent link="base_link"/>
@@ -223,6 +190,25 @@
     <origin xyz="0.1 0 0.17" rpy="0 0 0"/>
   </joint>
+  <link name="velodyne_mount">
+    <inertial>
+        <mass value="0.01" />
+        <origin xyz="0 0 0" />
+        <inertia ixx="0.001"  ixy="0.0"  ixz="0.0"
+        iyy="0.001"  iyz="0.0"
+            izz="0.001" />
+        </inertial>
+        <visual>
+            <geometry>
+                <box size="0.05 0.05 0.1" />
+            </geometry>
+        </visual>
+        <collision>
+            <geometry>
+                <box size="0.05 0.05 0.1" />
+            </geometry>
+        </collision>
+    </link>
   <xacro:VLP-16 parent="velodyne_mount" name="velodyne" topic="/velodyne_points" hz="10" organize_cloud="true" samples="200" gpu="false">
-    <origin xyz="0 0 0" rpy="0 0 0" />
+    <origin xyz="0.1 0 0.17" rpy="0 0 0"/>
   </xacro:VLP-16>
 </robot>
