Commit message: PGC-9 Feature Addition
Jackal Simulation configured with sensors and move base.

File: src/scout_mini_ros/jackal/jackal_description/urdf/accessories.urdf.xacro (robot description, xacro)
@@ -67,15 +67,15 @@
     - vlp16 (default)  :: Velodyne VLP16
   -->
-  <xacro:if value="$(optenv JACKAL_LASER_3D 0)">
+  <!-- <xacro:if value="$(optenv JACKAL_LASER_3D 0)"> -->
     <xacro:property name="lidar_3d_model" value="$(optenv JACKAL_LASER_3D_MODEL vlp16)" />
-    <xacro:if value="${lidar_3d_model == 'vlp16'}">
+    <!-- <xacro:if value="${lidar_3d_model == 'vlp16'}"> -->
       <xacro:vlp16_mount
           parent_link="$(optenv JACKAL_LASER_3D_MOUNT mid)_mount"
           prefix="$(optenv JACKAL_LASER_3D_MOUNT mid)"
-          topic="$(optenv JACKAL_LASER_3D_TOPIC mid/points)">
+          topic="$(optenv JACKAL_LASER_3D_TOPIC velodyne_points)">
         <origin xyz="$(optenv JACKAL_LASER_3D_OFFSET 0 0 0)" rpy="$(optenv JACKAL_LASER_3D_RPY 0 0 0)" />
       </xacro:vlp16_mount>
-    </xacro:if>
-  </xacro:if>
+    <!-- </xacro:if>
+  </xacro:if> -->
   <!-- If enabled, generate the upgraded Navsat payload (a Novatel Smart6). -->
   <xacro:if value="$(optenv JACKAL_NAVSAT 0)">
@@ -99,5 +99,5 @@
   <!-- Common camera mounts and accessory URDFs. -->
   <xacro:include filename="$(find jackal_description)/urdf/accessories/camera_mount.urdf.xacro" />
-  <xacro:include filename="$(find pointgrey_camera_description)/urdf/pointgrey_flea3.urdf.xacro" />
+  <xacro:include filename="$(find realsense2_description)/urdf/_d435.urdf.xacro" />
   <!-- If enabled, generate the flea3 camera payload with a tilt of 30 degrees. -->
   <xacro:if value="$(optenv JACKAL_FLEA3 0)">
@@ -110,5 +110,5 @@
       <child link="$(optenv JACKAL_FLEA3_MOUNT front)_camera_mount" />
     </joint>
-    <xacro:pointgrey_flea3 frame="$(optenv JACKAL_FLEA3_MOUNT front)_camera" name="$(optenv JACKAL_FLEA3_NAME front)"
+    <xacro:_d435 frame="$(optenv JACKAL_FLEA3_MOUNT front)_camera" name="$(optenv JACKAL_FLEA3_NAME front)"
       camera_x="0.0754" camera_y="0.029" camera_z="0.029"
       camera_mass="0.085" hfov="1.0471975512" fps="60" width="640" height="512"/>
@@ -122,5 +122,5 @@
   <!-- If enabled, generates a pair of flea3 cameras for stereo vision with a tilt of 30 degrees. -->
   <!-- Disabled temporarily due to metapackage issue. -->
-  <xacro:if value="$(optenv JACKAL_STEREO_FLEA3 0)">
+  <!-- <xacro:if value="$(optenv JACKAL_STEREO_FLEA3 0)">
     <xacro:stereo_camera_mount prefix="$(optenv JACKAL_FLEA3_MOUNT front)"
                        tilt="$(optenv JACKAL_FLEA3_TILT 0.5236)"/>
@@ -130,6 +130,6 @@
       <parent link="$(optenv JACKAL_FLEA3_MOUNT front)_mount" />
       <child link="$(optenv JACKAL_FLEA3_MOUNT front)_stereo_camera_mount" />
-    </joint>
-    <xacro:pointgrey_flea3 frame="$(optenv JACKAL_FLEA3_MOUNT front)_left_camera" name="$(optenv JACKAL_FLEA3_LEFT_NAME front/left)"
+    </joint> -->
+    <!-- <xacro:pointgrey_flea3 frame="$(optenv JACKAL_FLEA3_MOUNT front)_left_camera" name="$(optenv JACKAL_FLEA3_LEFT_NAME front/left)"
       camera_x="0.0754" camera_y="0.029" camera_z="0.029"
       camera_mass="0.085" hfov="1.0471975512" fps="60" width="640" height="512"/>
@@ -147,7 +147,10 @@
       <child link="$(optenv JACKAL_FLEA3_MOUNT front)_right_camera" />
     </joint>
-  </xacro:if>
+  </xacro:if> -->
   <!-- If enabled, generate the bumblebee2 camera payload with a tilt of 0 degrees. -->
-  <xacro:include filename="$(find pointgrey_camera_description)/urdf/pointgrey_bumblebee2.urdf.xacro" />
+  <xacro:include filename="$(find realsense2_description)/urdf/_d435.urdf.xacro" />
+  <xacro:sensor_d435 name="d435" parent="base_link">
+    <origin xyz="0.19 0 0.06" rpy="0 0 0"/>
+  </xacro:sensor_d435>
   <!-- If enabled, generate the bumblebee2 camera payload with a tilt of 0 degrees. -->
   <!-- Disabled temporarily due to metapackage issue. -->

File: src/scout_mini_ros/jackal/jackal_description/urdf/jackal.urdf.xacro (robot description, xacro)
@@ -241,5 +241,3 @@
   <!-- Optional custom includes. -->
   <xacro:include filename="$(optenv JACKAL_URDF_EXTRAS empty.urdf)" />
-  <!-- Optional for Clearpath internal softwares -->
-  <xacro:include filename="$(optenv CPR_URDF_EXTRAS empty.urdf)" />
 </robot>
